File: microstripline.kicad_pcb (KiCad board)
At the start: 2 copper layers, 304.8 x 304.8 mm, 11 parts

Commit message: 6.6mm幅完成
Parts:
- moved JP1 276.6 mm to (345.1, 238.8)
- moved TP2 10.2 mm to (340.4, 238.8)
- moved TP1 2.54 mm to (66.0, -35.6)
Connections:
- TP2 pad 1: GND -> Net-(JP1-A)
Routing:
- net Net-(JP1-A): track 1122.1 -> 10326.9 mm
- net GND: track 0.00 -> 11.6 mm, vias 0 -> 16
