File: 6.6mm_GAP/microstripline_6.6mm_gap.kicad_pcb (KiCad board)
At the start: 2 copper layers, 304.8 x 304.8 mm, 11 parts

Commit message: 条件をシルクで表示
Other:
- board text added: "全長:10.2m"
- board text added: "材質:FR-4 比誘電率:4.5 基板厚:0.6mm 箔厚:35μm 線幅:1.09mm 特性インピーダンス:50Ω"
- board text added: "電流伝搬速度計測基板"
