File: 6.6mm_GAP/microstripline_6.6mm_gap.kicad_pcb (KiCad board)
At the start: 2 copper layers, 304.8 x 304.8 mm, 11 parts

Commit message: [6.6mm]タイトル変更とシルク・ベタ位置調整
Other:
- board text added: "分布定数回路検証基板"
- board text removed: "電流伝搬速度計測基板"
